Commit message: REDO

File: src/scuttle_description/urdf/materials.xacro (robot description, xacro)
@@ -8,5 +8,8 @@
 </material>
 <material name="gray">
-  <color rgba="1.000 1.000 1.000 1.000"/>
+  <color rgba="0.500 0.500 0.500 1.000"/>
+</material>
+<material name="black">
+  <color rgba="0.000 0.000 0.000 1.000"/>
 </material>
 </robot>

File: src/scuttle_description/urdf/scuttle.xacro (robot description, xacro)
@@ -6,7 +6,7 @@
 <link name="base_link">
   <inertial>
-    <origin rpy="0 0 0" xyz="-1.166635410998978e-16 0.003797557168953781 0.01263544014076835"/>
-    <mass value="3.367819178653828"/>
-    <inertia ixx="0.061263" ixy="-0.0" ixz="-0.0" iyy="0.042394" iyz="-0.00082" izz="0.102286"/>
+    <origin rpy="0 0 0" xyz="-8.799632430808571e-17 -0.10062675010705613 0.08280154277913919"/>
+    <mass value="3.348734003283269"/>
+    <inertia ixx="0.060597" ixy="-0.0" ixz="-0.0" iyy="0.042291" iyz="-0.00058" izz="0.101721"/>
   </inertial>
   <visual>
@@ -24,12 +24,72 @@
   </collision>
 </link>
+<link name="lidar_base_1">
+  <inertial>
+    <origin rpy="0 0 0" xyz="1.2793131434440583e-17 -6.938893903907228e-18 0.028009771018959295"/>
+    <mass value="0.5065335084955669"/>
+    <inertia ixx="0.00039" ixy="0.0" ixz="0.0" iyy="0.00039" iyz="0.0" izz="0.000489"/>
+  </inertial>
+  <visual>
+    <origin rpy="0 0 0" xyz="-0.0 -0.03155 -0.09975"/>
+    <geometry>
+      <mesh filename="package://scuttle_description/meshes/lidar_base_1.stl" scale="0.001 0.001 0.001"/>
+    </geometry>
+    <material name="gray"/>
+  </visual>
+  <collision>
+    <origin rpy="0 0 0" xyz="-0.0 -0.03155 -0.09975"/>
+    <geometry>
+      <mesh filename="package://scuttle_description/meshes/lidar_base_1.stl" scale="0.001 0.001 0.001"/>
+    </geometry>
+  </collision>
+</link>
+<link name="lidar_top_1">
+  <inertial>
+    <origin rpy="0 0 0" xyz="2.173587506302513e-17 -2.7755575615628914e-17 0.009454772971040415"/>
+    <mass value="0.032608136404242656"/>
+    <inertia ixx="4e-06" ixy="-0.0" ixz="0.0" iyy="4e-06" iyz="-0.0" izz="6e-06"/>
+  </inertial>
+  <visual>
+    <origin rpy="0 0 0" xyz="-0.0 -0.03155 -0.16975"/>
+    <geometry>
+      <mesh filename="package://scuttle_description/meshes/lidar_top_1.stl" scale="0.001 0.001 0.001"/>
+    </geometry>
+    <material name="black"/>
+  </visual>
+  <collision>
+    <origin rpy="0 0 0" xyz="-0.0 -0.03155 -0.16975"/>
+    <geometry>
+      <mesh filename="package://scuttle_description/meshes/lidar_top_1.stl" scale="0.001 0.001 0.001"/>
+    </geometry>
+  </collision>
+</link>
+<link name="caster_1">
+  <inertial>
+    <origin rpy="0 0 0" xyz="0.0 -5.551115123125783e-17 -0.005625000000000017"/>
+    <mass value="0.019085175370557983"/>
+    <inertia ixx="1e-06" ixy="-0.0" ixz="-0.0" iyy="1e-06" iyz="0.0" izz="2e-06"/>
+  </inertial>
+  <visual>
+    <origin rpy="0 0 0" xyz="-0.0 0.2728 -0.015"/>
+    <geometry>
+      <mesh filename="package://scuttle_description/meshes/caster_1.stl" scale="0.001 0.001 0.001"/>
+    </geometry>
+    <material name="gray"/>
+  </visual>
+  <collision>
+    <origin rpy="0 0 0" xyz="-0.0 0.2728 -0.015"/>
+    <geometry>
+      <mesh filename="package://scuttle_description/meshes/caster_1.stl" scale="0.001 0.001 0.001"/>
+    </geometry>
+  </collision>
+</link>
 <link name="left_wheel_1">
   <inertial>
-    <origin rpy="0 0 0" xyz="0.03712499999999999 6.938893903907228e-17 1.734723475976807e-17"/>
+    <origin rpy="0 0 0" xyz="0.03712499999999999 3.552713678800501e-17 6.938893903907228e-18"/>
     <mass value="0.553600882889771"/>
     <inertia ixx="0.000476" ixy="0.0" ixz="0.0" iyy="0.000492" iyz="0.0" izz="0.000492"/>
   </inertial>
   <visual>
-    <origin rpy="0 0 0" xyz="-0.1524 -0.1054 0.028"/>
+    <origin rpy="0 0 0" xyz="-0.1524 -0.0 -0.04175"/>
     <geometry>
       <mesh filename="package://scuttle_description/meshes/left_wheel_1.stl" scale="0.001 0.001 0.001"/>
@@ -38,5 +98,5 @@
   </visual>
   <collision>
-    <origin rpy="0 0 0" xyz="-0.1524 -0.1054 0.028"/>
+    <origin rpy="0 0 0" xyz="-0.1524 -0.0 -0.04175"/>
     <geometry>
       <mesh filename="package://scuttle_description/meshes/left_wheel_1.stl" scale="0.001 0.001 0.001"/>
@@ -46,10 +106,10 @@
 <link name="right_wheel_1">
   <inertial>
-    <origin rpy="0 0 0" xyz="-0.037124999999999964 6.938893903907228e-17 1.734723475976807e-17"/>
+    <origin rpy="0 0 0" xyz="-0.037124999999999964 3.552713678800501e-17 2.0816681711721685e-17"/>
     <mass value="0.553600882889771"/>
     <inertia ixx="0.000476" ixy="-0.0" ixz="0.0" iyy="0.000492" iyz="0.0" izz="0.000492"/>
   </inertial>
   <visual>
-    <origin rpy="0 0 0" xyz="0.1524 -0.1054 0.028"/>
+    <origin rpy="0 0 0" xyz="0.1524 -0.0 -0.04175"/>
     <geometry>
       <mesh filename="package://scuttle_description/meshes/right_wheel_1.stl" scale="0.001 0.001 0.001"/>
@@ -58,5 +118,5 @@
   </visual>
   <collision>
-    <origin rpy="0 0 0" xyz="0.1524 -0.1054 0.028"/>
+    <origin rpy="0 0 0" xyz="0.1524 -0.0 -0.04175"/>
     <geometry>
       <mesh filename="package://scuttle_description/meshes/right_wheel_1.stl" scale="0.001 0.001 0.001"/>
@@ -64,42 +124,30 @@
   </collision>
 </link>
-<link name="lidar_1">
-  <inertial>
-    <origin rpy="0 0 0" xyz="1.2019382682516282e-17 2.7755575615628914e-17 0.031121245817537918"/>
-    <mass value="0.5391416448998095"/>
-    <inertia ixx="0.000475" ixy="0.0" ixz="0.0" iyy="0.000475" iyz="0.0" izz="0.000495"/>
-  </inertial>
-  <visual>
-    <origin rpy="0 0 0" xyz="-0.0 -0.13695 -0.03"/>
-    <geometry>
-      <mesh filename="package://scuttle_description/meshes/lidar_1.stl" scale="0.001 0.001 0.001"/>
-    </geometry>
-    <material name="gray"/>
-  </visual>
-  <collision>
-    <origin rpy="0 0 0" xyz="-0.0 -0.13695 -0.03"/>
-    <geometry>
-      <mesh filename="package://scuttle_description/meshes/lidar_1.stl" scale="0.001 0.001 0.001"/>
-    </geometry>
-  </collision>
-</link>
-<joint name="Rev4" type="continuous">
-  <origin rpy="0 0 0" xyz="0.1524 0.1054 -0.028"/>
+<joint name="Rigid1" type="fixed">
+  <origin rpy="0 0 0" xyz="0.0 0.03155 0.09975"/>
+  <parent link="base_link"/>
+  <child link="lidar_base_1"/>
+</joint>
+<joint name="Rigid2" type="fixed">
+  <origin rpy="0 0 0" xyz="0.0 0.0 0.07"/>
+  <parent link="lidar_base_1"/>
+  <child link="lidar_top_1"/>
+</joint>
+<joint name="Rigid3" type="fixed">
+  <origin rpy="0 0 0" xyz="0.0 -0.2728 0.015"/>
+  <parent link="base_link"/>
+  <child link="caster_1"/>
+</joint>
+<joint name="Rev1" type="continuous">
+  <origin rpy="0 0 0" xyz="0.1524 0.0 0.04175"/>
   <parent link="base_link"/>
   <child link="left_wheel_1"/>
   <axis xyz="1.0 0.0 0.0"/>
 </joint>
-<joint name="Rev5" type="continuous">
-  <origin rpy="0 0 0" xyz="-0.1524 0.1054 -0.028"/>
+<joint name="Rev2" type="continuous">
+  <origin rpy="0 0 0" xyz="-0.1524 0.0 0.04175"/>
   <parent link="base_link"/>
   <child link="right_wheel_1"/>
   <axis xyz="1.0 0.0 0.0"/>
 </joint>
-<joint name="Rigid6" type="fixed">
-  <origin rpy="0 0 -1.570796" xyz="0.0 0.13695 0.031"/>
-  <parent link="base_link"/>
-  <child link="lidar_1"/>
-  <!-- <axis xyz="-0.0 -0.13695 -0.01"/> -->
-  <!-- <axis xyz="0.0 0.0 0.0"/> -->
-</joint>
 </robot>

Commit message: SCUTTLE simulations

File: src/scuttle_description/urdf/materials.xacro (robot description, xacro)
@@ -4,12 +4,3 @@
   <color rgba="0.700 0.700 0.700 1.000"/>
 </material>
-<material name="blue">
-  <color rgba="0.100 0.100 0.700 1.000"/>
-</material>
-<material name="gray">
-  <color rgba="0.500 0.500 0.500 1.000"/>
-</material>
-<material name="black">
-  <color rgba="0.000 0.000 0.000 1.000"/>
-</material>
 </robot>

File: src/scuttle_description/urdf/scuttle.xacro (robot description, xacro)
@@ -6,7 +6,7 @@
 <link name="base_link">
   <inertial>
-    <origin rpy="0 0 0" xyz="-8.799632430808571e-17 -0.10062675010705613 0.08280154277913919"/>
-    <mass value="3.348734003283269"/>
-    <inertia ixx="0.060597" ixy="-0.0" ixz="-0.0" iyy="0.042291" iyz="-0.00058" izz="0.101721"/>
+    <origin rpy="0 0 0" xyz="2.12433370053547e-05 -0.07877992189559235 0.07392475478815927"/>
+    <mass value="3.288323846275119"/>
+    <inertia ixx="0.038876" ixy="1.3e-05" ixz="2e-06" iyy="0.047513" iyz="0.000485" izz="0.084083"/>
   </inertial>
   <visual>
@@ -24,130 +24,185 @@
   </collision>
 </link>
-<link name="lidar_base_1">
-  <inertial>
-    <origin rpy="0 0 0" xyz="1.2793131434440583e-17 -6.938893903907228e-18 0.028009771018959295"/>
-    <mass value="0.5065335084955669"/>
-    <inertia ixx="0.00039" ixy="0.0" ixz="0.0" iyy="0.00039" iyz="0.0" izz="0.000489"/>
-  </inertial>
-  <visual>
-    <origin rpy="0 0 0" xyz="-0.0 -0.03155 -0.09975"/>
-    <geometry>
-      <mesh filename="package://scuttle_description/meshes/lidar_base_1.stl" scale="0.001 0.001 0.001"/>
-    </geometry>
-    <material name="gray"/>
-  </visual>
-  <collision>
-    <origin rpy="0 0 0" xyz="-0.0 -0.03155 -0.09975"/>
-    <geometry>
-      <mesh filename="package://scuttle_description/meshes/lidar_base_1.stl" scale="0.001 0.001 0.001"/>
-    </geometry>
-  </collision>
-</link>
-<link name="lidar_top_1">
-  <inertial>
-    <origin rpy="0 0 0" xyz="2.173587506302513e-17 -2.7755575615628914e-17 0.009454772971040415"/>
-    <mass value="0.032608136404242656"/>
-    <inertia ixx="4e-06" ixy="-0.0" ixz="0.0" iyy="4e-06" iyz="-0.0" izz="6e-06"/>
-  </inertial>
-  <visual>
-    <origin rpy="0 0 0" xyz="-0.0 -0.03155 -0.16975"/>
-    <geometry>
-      <mesh filename="package://scuttle_description/meshes/lidar_top_1.stl" scale="0.001 0.001 0.001"/>
-    </geometry>
-    <material name="black"/>
-  </visual>
-  <collision>
-    <origin rpy="0 0 0" xyz="-0.0 -0.03155 -0.16975"/>
-    <geometry>
-      <mesh filename="package://scuttle_description/meshes/lidar_top_1.stl" scale="0.001 0.001 0.001"/>
-    </geometry>
-  </collision>
-</link>
-<link name="caster_1">
-  <inertial>
-    <origin rpy="0 0 0" xyz="0.0 -5.551115123125783e-17 -0.005625000000000017"/>
-    <mass value="0.019085175370557983"/>
-    <inertia ixx="1e-06" ixy="-0.0" ixz="-0.0" iyy="1e-06" iyz="0.0" izz="2e-06"/>
-  </inertial>
-  <visual>
-    <origin rpy="0 0 0" xyz="-0.0 0.2728 -0.015"/>
-    <geometry>
-      <mesh filename="package://scuttle_description/meshes/caster_1.stl" scale="0.001 0.001 0.001"/>
-    </geometry>
-    <material name="gray"/>
-  </visual>
-  <collision>
-    <origin rpy="0 0 0" xyz="-0.0 0.2728 -0.015"/>
-    <geometry>
-      <mesh filename="package://scuttle_description/meshes/caster_1.stl" scale="0.001 0.001 0.001"/>
-    </geometry>
-  </collision>
-</link>
-<link name="left_wheel_1">
-  <inertial>
-    <origin rpy="0 0 0" xyz="0.03712499999999999 3.552713678800501e-17 6.938893903907228e-18"/>
-    <mass value="0.553600882889771"/>
-    <inertia ixx="0.000476" ixy="0.0" ixz="0.0" iyy="0.000492" iyz="0.0" izz="0.000492"/>
-  </inertial>
-  <visual>
-    <origin rpy="0 0 0" xyz="-0.1524 -0.0 -0.04175"/>
-    <geometry>
-      <mesh filename="package://scuttle_description/meshes/left_wheel_1.stl" scale="0.001 0.001 0.001"/>
-    </geometry>
-    <material name="blue"/>
-  </visual>
-  <collision>
-    <origin rpy="0 0 0" xyz="-0.1524 -0.0 -0.04175"/>
-    <geometry>
-      <mesh filename="package://scuttle_description/meshes/left_wheel_1.stl" scale="0.001 0.001 0.001"/>
-    </geometry>
-  </collision>
-</link>
-<link name="right_wheel_1">
-  <inertial>
-    <origin rpy="0 0 0" xyz="-0.037124999999999964 3.552713678800501e-17 2.0816681711721685e-17"/>
-    <mass value="0.553600882889771"/>
-    <inertia ixx="0.000476" ixy="-0.0" ixz="0.0" iyy="0.000492" iyz="0.0" izz="0.000492"/>
-  </inertial>
-  <visual>
-    <origin rpy="0 0 0" xyz="0.1524 -0.0 -0.04175"/>
-    <geometry>
-      <mesh filename="package://scuttle_description/meshes/right_wheel_1.stl" scale="0.001 0.001 0.001"/>
-    </geometry>
-    <material name="blue"/>
-  </visual>
-  <collision>
-    <origin rpy="0 0 0" xyz="0.1524 -0.0 -0.04175"/>
-    <geometry>
-      <mesh filename="package://scuttle_description/meshes/right_wheel_1.stl" scale="0.001 0.001 0.001"/>
-    </geometry>
-  </collision>
-</link>
-<joint name="Rigid1" type="fixed">
-  <origin rpy="0 0 0" xyz="0.0 0.03155 0.09975"/>
-  <parent link="base_link"/>
-  <child link="lidar_base_1"/>
-</joint>
-<joint name="Rigid2" type="fixed">
-  <origin rpy="0 0 0" xyz="0.0 0.0 0.07"/>
-  <parent link="lidar_base_1"/>
-  <child link="lidar_top_1"/>
-</joint>
-<joint name="Rigid3" type="fixed">
-  <origin rpy="0 0 0" xyz="0.0 -0.2728 0.015"/>
-  <parent link="base_link"/>
-  <child link="caster_1"/>
-</joint>
-<joint name="Rev1" type="continuous">
-  <origin rpy="0 0 0" xyz="0.1524 0.0 0.04175"/>
-  <parent link="base_link"/>
-  <child link="left_wheel_1"/>
-  <axis xyz="1.0 0.0 0.0"/>
-</joint>
-<joint name="Rev2" type="continuous">
-  <origin rpy="0 0 0" xyz="-0.1524 0.0 0.04175"/>
-  <parent link="base_link"/>
-  <child link="right_wheel_1"/>
-  <axis xyz="1.0 0.0 0.0"/>
+<link name="l_wheel_1">
+  <inertial>
+    <origin rpy="0 0 0" xyz="-0.020325481156161784 -9.763736334427187e-09 4.516951403188418e-09"/>
+    <mass value="0.5928646271111422"/>
+    <inertia ixx="0.000334" ixy="0.0" ixz="-0.0" iyy="0.000332" iyz="-0.0" izz="0.000332"/>
+  </inertial>
+  <visual>
+    <origin rpy="0 0 0" xyz="-0.21235 -0.0 -0.04175"/>
+    <geometry>
+      <mesh filename="package://scuttle_description/meshes/l_wheel_1.stl" scale="0.001 0.001 0.001"/>
+    </geometry>
+    <material name="silver"/>
+  </visual>
+  <collision>
+    <origin rpy="0 0 0" xyz="-0.21235 -0.0 -0.04175"/>
+    <geometry>
+      <mesh filename="package://scuttle_description/meshes/l_wheel_1.stl" scale="0.001 0.001 0.001"/>
+    </geometry>
+  </collision>
+</link>
+<link name="r_wheel_1">
+  <inertial>
+    <origin rpy="0 0 0" xyz="0.020325563043213257 1.3954236146756306e-08 2.0353343177514915e-09"/>
+    <mass value="0.592867092340216"/>
+    <inertia ixx="0.000334" ixy="0.0" ixz="0.0" iyy="0.000332" iyz="-0.0" izz="0.000332"/>
+  </inertial>
+  <visual>
+    <origin rpy="0 0 0" xyz="0.21215 0.0 -0.04175"/>
+    <geometry>
+      <mesh filename="package://scuttle_description/meshes/r_wheel_1.stl" scale="0.001 0.001 0.001"/>
+    </geometry>
+    <material name="silver"/>
+  </visual>
+  <collision>
+    <origin rpy="0 0 0" xyz="0.21215 0.0 -0.04175"/>
+    <geometry>
+      <mesh filename="package://scuttle_description/meshes/r_wheel_1.stl" scale="0.001 0.001 0.001"/>
+    </geometry>
+  </collision>
+</link>
+<link name="LiDAR_1">
+  <inertial>
+    <origin rpy="0 0 0" xyz="-0.0010241190327231165 -0.0008953477993804172 0.009594767416774092"/>
+    <mass value="0.07327266108520486"/>
+    <inertia ixx="2.5e-05" ixy="1e-06" ixz="0.0" iyy="2.5e-05" iyz="0.0" izz="4.4e-05"/>
+  </inertial>
+  <visual>
+    <origin rpy="0 0 0" xyz="-0.0 0.0275 -0.1096"/>
+    <geometry>
+      <mesh filename="package://scuttle_description/meshes/LiDAR_1.stl" scale="0.001 0.001 0.001"/>
+    </geometry>
+    <material name="silver"/>
+  </visual>
+  <collision>
+    <origin rpy="0 0 0" xyz="-0.0 0.0275 -0.1096"/>
+    <geometry>
+      <mesh filename="package://scuttle_description/meshes/LiDAR_1.stl" scale="0.001 0.001 0.001"/>
+    </geometry>
+  </collision>
+</link>
+<link name="r_caster_swivel_1">
+  <inertial>
+    <origin rpy="0 0 0" xyz="-0.0002554502352885568 0.010633952722858359 -0.012968467515129908"/>
+    <mass value="0.02074189648802402"/>
+    <inertia ixx="7e-06" ixy="0.0" ixz="0.0" iyy="8e-06" iyz="1e-06" izz="9e-06"/>
+  </inertial>
+  <visual>
+    <origin rpy="0 0 0" xyz="0.119279 0.254415 -0.059282"/>
+    <geometry>
+      <mesh filename="package://scuttle_description/meshes/r_caster_swivel_1.stl" scale="0.001 0.001 0.001"/>
+    </geometry>
+    <material name="silver"/>
+  </visual>
+  <collision>
+    <origin rpy="0 0 0" xyz="0.119279 0.254415 -0.059282"/>
+    <geometry>
+      <mesh filename="package://scuttle_description/meshes/r_caster_swivel_1.stl" scale="0.001 0.001 0.001"/>
+    </geometry>
+  </collision>
+</link>
+<link name="l_caster_swivel_1">
+  <inertial>
+    <origin rpy="0 0 0" xyz="-0.00025520971284771765 0.010633952722903461 -0.012968467515129777"/>
+    <mass value="0.02074189648802399"/>
+    <inertia ixx="7e-06" ixy="0.0" ixz="0.0" iyy="8e-06" iyz="1e-06" izz="9e-06"/>
+  </inertial>
+  <visual>
+    <origin rpy="0 0 0" xyz="-0.119015 0.254415 -0.059282"/>
+    <geometry>
+      <mesh filename="package://scuttle_description/meshes/l_caster_swivel_1.stl" scale="0.001 0.001 0.001"/>
+    </geometry>
+    <material name="silver"/>
+  </visual>
+  <collision>
+    <origin rpy="0 0 0" xyz="-0.119015 0.254415 -0.059282"/>
+    <geometry>
+      <mesh filename="package://scuttle_description/meshes/l_caster_swivel_1.stl" scale="0.001 0.001 0.001"/>
+    </geometry>
+  </collision>
+</link>
+<link name="l_caster_wheel_1">
+  <inertial>
+    <origin rpy="0 0 0" xyz="0.0160002016389222 -1.6368916427866864e-07 -7.02880924990934e-08"/>
+    <mass value="0.03841110590847018"/>
+    <inertia ixx="1.2e-05" ixy="0.0" ixz="-0.0" iyy="7e-06" iyz="0.0" izz="7e-06"/>
+  </inertial>
+  <visual>
+    <origin rpy="0 0 0" xyz="-0.101223 0.230415 -0.025282"/>
+    <geometry>
+      <mesh filename="package://scuttle_description/meshes/l_caster_wheel_1.stl" scale="0.001 0.001 0.001"/>
+    </geometry>
+    <material name="silver"/>
+  </visual>
+  <collision>
+    <origin rpy="0 0 0" xyz="-0.101223 0.230415 -0.025282"/>
+    <geometry>
+      <mesh filename="package://scuttle_description/meshes/l_caster_wheel_1.stl" scale="0.001 0.001 0.001"/>
+    </geometry>
+  </collision>
+</link>
+<link name="r_caster_wheel_1">
+  <inertial>
+    <origin rpy="0 0 0" xyz="-0.016000038883518655 -1.6368920854881175e-07 -7.028809271419911e-08"/>
+    <mass value="0.03841110590847031"/>
+    <inertia ixx="1.2e-05" ixy="-0.0" ixz="0.0" iyy="7e-06" iyz="0.0" izz="7e-06"/>
+  </inertial>
+  <visual>
+    <origin rpy="0 0 0" xyz="0.105071 0.230415 -0.025282"/>
+    <geometry>
+      <mesh filename="package://scuttle_description/meshes/r_caster_wheel_1.stl" scale="0.001 0.001 0.001"/>
+    </geometry>
+    <material name="silver"/>
+  </visual>
+  <collision>
+    <origin rpy="0 0 0" xyz="0.105071 0.230415 -0.025282"/>
+    <geometry>
+      <mesh filename="package://scuttle_description/meshes/r_caster_wheel_1.stl" scale="0.001 0.001 0.001"/>
+    </geometry>
+  </collision>
+</link>
+<joint name="l_wheel_joint" type="continuous">
+  <origin rpy="0 0 0" xyz="0.21235 0.0 0.04175"/>
+  <parent link="base_link"/>
+  <child link="l_wheel_1"/>
+  <axis xyz="1.0 -0.0 0.0"/>
+</joint>
+<joint name="r_wheel_joint" type="continuous">
+  <origin rpy="0 0 0" xyz="-0.21215 0.0 0.04175"/>
+  <parent link="base_link"/>
+  <child link="r_wheel_1"/>
+  <axis xyz="1.0 0.0 -0.0"/>
+</joint>
+<joint name="lidar" type="continuous">
+  <origin rpy="0 0 0" xyz="0.0 -0.0275 0.1096"/>
+  <parent link="base_link"/>
+  <child link="LiDAR_1"/>
+  <axis xyz="0.0 0.0 1.0"/>
+</joint>
+<joint name="r_caster_swivel_joint" type="continuous">
+  <origin rpy="0 0 0" xyz="-0.119279 -0.254415 0.059282"/>
+  <parent link="base_link"/>
+  <child link="r_caster_swivel_1"/>
+  <axis xyz="0.0 0.0 1.0"/>
+</joint>
+<joint name="l_caster_swivel_joint" type="continuous">
+  <origin rpy="0 0 0" xyz="0.119015 -0.254415 0.059282"/>
+  <parent link="base_link"/>
+  <child link="l_caster_swivel_1"/>
+  <axis xyz="0.0 -0.0 1.0"/>
+</joint>
+<joint name="r_caster_wheel_joint" type="continuous">
+  <origin rpy="0 0 0" xyz="-0.017792 0.024 -0.034"/>
+  <parent link="l_caster_swivel_1"/>
+  <child link="l_caster_wheel_1"/>
+  <axis xyz="1.0 0.0 -0.0"/>
+</joint>
+<joint name="l_caster_wheel_joint" type="continuous">
+  <origin rpy="0 0 0" xyz="0.014208 0.024 -0.034"/>
+  <parent link="r_caster_swivel_1"/>
+  <child link="r_caster_wheel_1"/>
+  <axis xyz="-1.0 -0.0 0.0"/>
 </joint>
 </robot>
