Commit message: mapping rviz error with lidar and base_link

File: src/scuttle_description/urdf/scuttle.xacro (robot description, xacro)
@@ -100,4 +100,6 @@
   <parent link="base_link"/>
   <child link="lidar_1"/>
+  <!-- <axis xyz="-0.0 -0.13695 -0.01"/> -->
+  <!-- <axis xyz="0.0 0.0 0.0"/> -->
 </joint>
 </robot>

Commit message: linked lidar with scuttle xacro

File: src/scuttle_description/urdf/scuttle.xacro (robot description, xacro)
@@ -176,6 +176,6 @@
   <axis xyz="1.0 0.0 -0.0"/>
 </joint>
-<joint name="lidar" type="continuous">
-  <origin rpy="0 0 0" xyz="0.0 -0.0275 0.1096"/>
+<joint name="lidar" type="fixed">
+  <origin rpy="0 0 1.570796" xyz="0.0 -0.0275 0.1096"/>
   <parent link="base_link"/>
   <child link="LiDAR_1"/>

Commit message: added scuttle_description as git repo

File: src/scuttle_description/urdf/scuttle.xacro (robot description, xacro)
@@ -177,5 +177,5 @@
 </joint>
 <joint name="lidar" type="fixed">
-  <origin rpy="0 0 1.570796" xyz="0.0 -0.0275 0.1096"/>
+  <origin rpy="0 0 0" xyz="0.0 -0.0275 0.1096"/>
   <parent link="base_link"/>
   <child link="LiDAR_1"/>
